File: board/universalStepDown.sch (KiCad schematic (older format))
At the start: 15 parts, among them J1 IO, U1 SY8105

Commit message: Fix issues by cednik, prepare multi-voltage variant
Parts:
- C2: footprint Capacitor_SMD:C_0402_1005Metric -> Capacitor_SMD:C_0603_1608Metric; LCSC C1525 -> C14663
- R2: value 27k -> 27k (for 5V)/44.2k (for 3V3); LCSC C25771 -> (none); LCSC_3V3 (none) -> C25895; LCSC_5V5 (none) -> C25771
- R3: value 47k -> 1M; LCSC C25792 -> C26083
Connections:
- net +5V renamed VOUT
Other:
- moved on the sheet: C3, C4, C6
Changed lines of the file:
@@
 P 6250 4500
 F 0 "R2" H 6320 4546 50  0000 L CNN
-F 1 "27k" H 6320 4455 50  0000 L CNN
+F 1 "27k (for 5V)/44.2k (for 3V3)" H 6320 4455 50  0000 L CNN
 F 2 "Resistor_SMD:R_0402_1005Metric" V 6180 4500 50  0001 C CNN
 F 3 "~" H 6250 4500 50  0001 C CNN
-F 4 "C25771" H 6250 4500 50  0001 C CNN "LCSC"
+F 4 "C25771" H 6250 4500 50  0001 C CNN "LCSC_5V5"
+F 5 "C25895" H 6250 4500 50  0001 C CNN "LCSC_3V3"
 	1    6250 4500
 	1    0    0    -1
@@
 $EndComp
 $Comp
-L power:+5V #PWR04
-U 1 1 5F1387C7
-P 7950 3750
-F 0 "#PWR04" H 7950 3600 50  0001 C CNN
-F 1 "+5V" H 7965 3923 50  0000 C CNN
-F 2 "" H 7950 3750 50  0001 C CNN
-F 3 "" H 7950 3750 50  0001 C CNN
-	1    7950 3750
-	0    1    1    0
-$EndComp
-$Comp
 L power:GND #PWR02
 U 1 1 5F13A365
@@
 F 0 "C2" V 5398 3500 50  0000 C CNN
 F 1 "100n" V 5489 3500 50  0000 C CNN
-F 2 "Capacitor_SMD:C_0402_1005Metric" H 5688 3350 50  0001 C CNN
+F 2 "Capacitor_SMD:C_0603_1608Metric" H 5688 3350 50  0001 C CNN
 F 3 "~" H 5650 3500 50  0001 C CNN
-F 4 "C1525" H 5650 3500 50  0001 C CNN "LCSC"
+F 4 "C14663" H 5650 3500 50  0001 C CNN "LCSC"
 	1    5650 3500
 	0    1    1    0
@@
 L Device:C C3
 U 1 1 5F13FA3D
-P 6650 4000
-F 0 "C3" H 6535 3954 50  0000 R CNN
-F 1 "47p" H 6535 4045 50  0000 R CNN
-F 2 "Capacitor_SMD:C_0402_1005Metric" H 6688 3850 50  0001 C CNN
-F 3 "~" H 6650 4000 50  0001 C CNN
-F 4 "C1567" H 6650 4000 50  0001 C CNN "LCSC"
-	1    6650 4000
+P 8050 4000
+F 0 "C3" H 7935 3954 50  0000 R CNN
+F 1 "47p" H 7935 4045 50  0000 R CNN
+F 2 "Capacitor_SMD:C_0402_1005Metric" H 8088 3850 50  0001 C CNN
+F 3 "~" H 8050 4000 50  0001 C CNN
+F 4 "C1567" H 8050 4000 50  0001 C CNN "LCSC"
+	1    8050 4000
 	-1   0    0    1
 $EndComp
@@
 L Device:C C4
 U 1 1 5F14017E
-P 7100 4000
-F 0 "C4" H 6985 3954 50  0000 R CNN
-F 1 "22u" H 6985 4045 50  0000 R CNN
-F 2 "Capacitor_SMD:C_0805_2012Metric" H 7138 3850 50  0001 C CNN
-F 3 "~" H 7100 4000 50  0001 C CNN
-F 4 "C45783" H 7100 4000 50  0001 C CNN "LCSC"
-	1    7100 4000
+P 8500 4000
+F 0 "C4" H 8385 3954 50  0000 R CNN
+F 1 "22u" H 8385 4045 50  0000 R CNN
+F 2 "Capacitor_SMD:C_0805_2012Metric" H 8538 3850 50  0001 C CNN
+F 3 "~" H 8500 4000 50  0001 C CNN
+F 4 "C45783" H 8500 4000 50  0001 C CNN "LCSC"
+	1    8500 4000
 	-1   0    0    1
 $EndComp
@@
 L power:GND #PWR05
 U 1 1 5F140637
-P 7100 4300
-F 0 "#PWR05" H 7100 4050 50  0001 C CNN
-F 1 "GND" H 7105 4127 50  0000 C CNN
-F 2 "" H 7100 4300 50  0001 C CNN
-F 3 "" H 7100 4300 50  0001 C CNN
-	1    7100 4300
-	1    0    0    -1
-$EndComp
-Wire Wire Line
-	7100 4150 7100 4300
+P 8500 4300
+F 0 "#PWR05" H 8500 4050 50  0001 C CNN
+F 1 "GND" H 8505 4127 50  0000 C CNN
+F 2 "" H 8500 4300 50  0001 C CNN
+F 3 "" H 8500 4300 50  0001 C CNN
+	1    8500 4300
+	1    0    0    -1
+$EndComp
+Wire Wire Line
+	8500 4150 8500 4300
 Wire Wire Line
 	6250 3750 6650 3750
 Wire Wire Line
-	6650 3750 6650 3850
+	8050 3750 8050 3850
 Connection ~ 6250 3750
 Wire Wire Line
-	6650 4150 6650 4250
-Wire Wire Line
-	6650 4250 6250 4250
-Wire Wire Line
-	6650 3750 7100 3750
-Wire Wire Line
-	7100 3750 7100 3850
+	8050 4150 8050 4250
+Wire Wire Line
+	8500 3750 8500 3850
 Connection ~ 6650 3750
-Connection ~ 7100 3750
 $Comp
 L Device:R R3
@@
 P 4900 4000
 F 0 "R3" H 4970 4046 50  0000 L CNN
-F 1 "47k" H 4970 3955 50  0000 L CNN
+F 1 "1M" H 4970 3955 50  0000 L CNN
 F 2 "Resistor_SMD:R_0402_1005Metric" V 4830 4000 50  0001 C CNN
 F 3 "~" H 4900 4000 50  0001 C CNN
-F 4 "C25792" H 4900 4000 50  0001 C CNN "LCSC"
+F 4 "C26083" H 4900 4000 50  0001 C CNN "LCSC"
 	1    4900 4000
 	1    0    0    -1
@@
 $EndComp
 $Comp
-L power:+5V #PWR06
-U 1 1 5F120EBB
-P 6450 1850
-F 0 "#PWR06" H 6450 1700 50  0001 C CNN
-F 1 "+5V" H 6465 2023 50  0000 C CNN
-F 2 "" H 6450 1850 50  0001 C CNN
-F 3 "" H 6450 1850 50  0001 C CNN
-	1    6450 1850
-	1    0    0    -1
-$EndComp
-$Comp
 L power:GND #PWR07
 U 1 1 5F12144C
@@
 Connection ~ 4900 4250
 $Comp
-L power:+5V #PWR0102
-U 1 1 5F5785E6
-P 4900 2350
-F 0 "#PWR0102" H 4900 2200 50  0001 C CNN
-F 1 "+5V" H 4915 2523 50  0000 C CNN
-F 2 "" H 4900 2350 50  0001 C CNN
-F 3 "" H 4900 2350 50  0001 C CNN
-	1    4900 2350
-	0    -1   -1   0
-$EndComp
-$Comp
 L power:VCC #PWR0103
 U 1 1 5F578D79
@@
 L Device:C C6
 U 1 1 5F58A9EB
-P 7600 4000
-F 0 "C6" H 7485 3954 50  0000 R CNN
-F 1 "22u" H 7485 4045 50  0000 R CNN
-F 2 "Capacitor_SMD:C_0805_2012Metric" H 7638 3850 50  0001 C CNN
-F 3 "~" H 7600 4000 50  0001 C CNN
-F 4 "C45783" H 7600 4000 50  0001 C CNN "LCSC"
-	1    7600 4000
+P 9000 4000
+F 0 "C6" H 8885 3954 50  0000 R CNN
+F 1 "22u" H 8885 4045 50  0000 R CNN
+F 2 "Capacitor_SMD:C_0805_2012Metric" H 9038 3850 50  0001 C CNN
+F 3 "~" H 9000 4000 50  0001 C CNN
+F 4 "C45783" H 9000 4000 50  0001 C CNN "LCSC"
+	1    9000 4000
 	-1   0    0    1
 $EndComp
 Wire Wire Line
-	7100 3750 7600 3750
-Wire Wire Line
-	7600 3750 7600 3850
-Wire Wire Line
-	7600 4150 7600 4300
+	9000 3750 9000 3850
+Wire Wire Line
+	9000 4150 9000 4300
 $Comp
 L power:GND #PWR0105
 U 1 1 5F58C152
-P 7600 4300
-F 0 "#PWR0105" H 7600 4050 50  0001 C CNN
-F 1 "GND" H 7605 4127 50  0000 C CNN
-F 2 "" H 7600 4300 50  0001 C CNN
-F 3 "" H 7600 4300 50  0001 C CNN
-	1    7600 4300
-	1    0    0    -1
-$EndComp
-Wire Wire Line
-	7600 3750 7950 3750
-Connection ~ 7600 3750
+P 9000 4300
+F 0 "#PWR0105" H 9000 4050 50  0001 C CNN
+F 1 "GND" H 9005 4127 50  0000 C CNN
+F 2 "" H 9000 4300 50  0001 C CNN
+F 3 "" H 9000 4300 50  0001 C CNN
+	1    9000 4300
+	1    0    0    -1
+$EndComp
 Text Label 5950 4250 0    50   ~ 0
 FB
@@
 Wire Wire Line
 	4200 2250 4100 2250
+Text GLabel 9400 3750 2    50   Input ~ 0
+VOUT
+Text GLabel 4900 2350 0    50   Input ~ 0
+VOUT
+Connection ~ 8050 3750
+Wire Wire Line
+	8050 3750 8500 3750
+Connection ~ 8500 3750
+Wire Wire Line
+	8500 3750 9000 3750
+Connection ~ 9000 3750
+Wire Wire Line
+	9000 3750 9400 3750
+Wire Wire Line
+	6650 3750 8050 3750
+Wire Wire Line
+	6250 4250 8050 4250
+Text GLabel 6450 1850 1    50   Input ~ 0
+VOUT
 $EndSCHEMATC

Commit message: Prepare Makefile
Parts:
- J1: footprint Connector_PinHeader_2.54mm:PinHeader_1x04_P2.54mm_Horizontal -> universalStepDown:PinHeader_1x04_P2.54mm_Horizontal
- R2: LCSC_5V (none) -> C25771; LCSC_5V5 C25771 -> (none)
Changed lines of the file:
@@
 F 2 "Resistor_SMD:R_0402_1005Metric" V 6180 4500 50  0001 C CNN
 F 3 "~" H 6250 4500 50  0001 C CNN
-F 4 "C25771" H 6250 4500 50  0001 C CNN "LCSC_5V5"
+F 4 "C25771" H 6250 4500 50  0001 C CNN "LCSC_5V"
 F 5 "C25895" H 6250 4500 50  0001 C CNN "LCSC_3V3"
 	1    6250 4500
@@
 F 0 "J1" H 5180 2142 50  0000 L CNN
 F 1 "IO" H 5180 2051 50  0000 L CNN
-F 2 "Connector_PinHeader_2.54mm:PinHeader_1x04_P2.54mm_Horizontal" H 5100 2150 50  0001 C CNN
+F 2 "universalStepDown:PinHeader_1x04_P2.54mm_Horizontal" H 5100 2150 50  0001 C CNN
 F 3 "~" H 5100 2150 50  0001 C CNN
 	1    5100 2150
